File: RP2350A_dev_board.kicad_sch (KiCad schematic)
At the start: 52 parts, among them J1 Debug Headers, J2 USB_C_Female_USB2.0_16P, J3 I2C Headers, SW1 Button, SW2 Bootstrap, U1 USBLC6-2SC6, U2 SPX3819M5-L-3-3, U3 RP2350A, U4 W25Q128JVS, Y2 12MHz Crystal GND2,4

Commit message: Replaced +1V1 and +3V3 planes with wide routes. Routed all power. Finished all routing.
Connections:
- net USB_DM renamed USB_DN
Changed lines of the file:
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@@
 		)
 	)
-	(label "USB_DM"
+	(label "USB_DN"
 		(at 81.28 162.56 180)
 		(effects
@@
 		)
 	)
-	(label "USB_DM"
+	(label "USB_DN"
 		(at 208.28 92.71 180)
 		(effects

Commit message: Finished routing. Cleared ERC on schematic and layout.
Parts:
- U3: symbol custom:RP2350A -> custom:RP2350A_custom
Changed lines of the file:
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@@
 	)
 	(symbol
-		(lib_id "custom:RP2350A")
+		(lib_id "custom:RP2350A_custom")
 		(at 111.76 59.69 0)
 		(unit 1)

Commit message: Final commit for time being, getting board printed and assembled was outside my price range. Unfortunately, oldering 0604 components is also outside my skill range. Project needs to be reorganized using through-hole components.
Parts:
- J1, J3: now left out of the parts list
- R4, R5: JLCPCB Part Number C177401 -> (none); LCSC Part Number (none) -> C177401; Manfacturer Part Number RCT0327RJLF -> (none); Manufacturer Part Number (none) -> RCT0327RJLF
- U1: Distributor Link 1 (none) -> https://www.mouser.com/ProductDetail/STMicroelectronics/USB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; Distributor Link 2 (none) -> https://www.digikey.com/en/products/detail/stmicroelectroni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; LCSC Part Number (none) -> C7519; Manufacturer (none) -> STMicroelectronics; Manufacturer Part Number (none) -> USBLC6-2SC6
- U2: Distributor Link 1 (none) -> https://www.mouser.com/ProductDetail/MaxLinear/SPX3819M5-L-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; Distributor Link 2 (none) -> https://www.digikey.com/en/products/detail/maxlinear-inc/SP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; LCSC Part Number (none) -> C20617301; Manufacturer (none) -> TECH PUBLIC; Manufacturer Part Number (none) -> SPX3819M5-L-3-3
